File: din_meter_atm90e26.sch (KiCad schematic (older format))
At the start: 61 parts, among them J1 USEL, J2 MMD1, J3 MMD0, J4 CONN_02X18, J5 CONN_01X10, J6 USEL, J7 MMD1, J8 MMD0, M1 ATM90E26_ATM90E26, M2 ATM90E26_ATM90E26, Y1 Crystal_Small, Y2 Crystal_Small

Commit message: First pass at layout.
Parts:
- removed C21, C22, C23, C24: 33n, Capacitors_SMD:C_0402, symbol C_Small
- removed CF1_0: CF1_0, Measurement_Points:Measurement_Point_Round-SMD-Pad_Small, symbol TEST_1P
- removed CF1_1: CF1_1, Measurement_Points:Measurement_Point_Round-SMD-Pad_Small, symbol TEST_1P
- removed CF2_0: CF2_0, Measurement_Points:Measurement_Point_Round-SMD-Pad_Small, symbol TEST_1P
- removed CF2_1: CF2_1, Measurement_Points:Measurement_Point_Round-SMD-Pad_Small, symbol TEST_1P
- removed IRQ_0: IRQ_0, Measurement_Points:Measurement_Point_Round-SMD-Pad_Small, symbol TEST_1P
- removed IRQ_1: IRQ_1, Measurement_Points:Measurement_Point_Round-SMD-Pad_Small, symbol TEST_1P
- removed J1, J6: USEL, Connectors:GS3, symbol GS3
- removed J2, J7: MMD1, Connectors:GS3, symbol GS3
- removed J3, J8: MMD0, Connectors:GS3, symbol GS3
- removed J4: CONN_02X18, Connectors:PCI-EXPRESS, symbol PCIx1
- removed LOGO1: Logo_Open_Hardware_Small, Symbols:OSHW-Logo2_7.3x6mm_SilkScreen, symbol Logo_Open_Hardware_Small
- removed R10, R7, R8, R9: 1K, Resistors_SMD:R_0402, symbol R_Small
- removed WARN_0: WARN_0, Measurement_Points:Measurement_Point_Round-SMD-Pad_Small, symbol TEST_1P
- removed WARN_1: WARN_1, Measurement_Points:Measurement_Point_Round-SMD-Pad_Small, symbol TEST_1P
- removed ZX_0: ZX_0, Measurement_Points:Measurement_Point_Round-SMD-Pad_Small, symbol TEST_1P
- removed ZX_1: ZX_1, Measurement_Points:Measurement_Point_Round-SMD-Pad_Small, symbol TEST_1P
- added J1: PCIx1, Connectors:PCI-EXPRESS, symbol din_meter_atm90e26-rescue:PCIx1
- added J2: Conn_01x05, FitHome_conn:conn_5_2.54mm, symbol conn:Conn_01x05
- added TP_I1N_0: I1N_0, MeasurementPoints:Measurement_Point_Round-SMD-Pad_Small, symbol conn:TEST_1P
- added TP_I1N_1: I1N_1, MeasurementPoints:Measurement_Point_Round-SMD-Pad_Small, symbol conn:TEST_1P
- added TP_I1P_0: I1P_0, MeasurementPoints:Measurement_Point_Round-SMD-Pad_Small, symbol conn:TEST_1P
- added TP_I1P_1: I1P_1, MeasurementPoints:Measurement_Point_Round-SMD-Pad_Small, symbol conn:TEST_1P
- added TP_VN_0: VN_0, MeasurementPoints:Measurement_Point_Round-SMD-Pad_Small, symbol conn:TEST_1P
- added TP_VN_1: VN_1, MeasurementPoints:Measurement_Point_Round-SMD-Pad_Small, symbol conn:TEST_1P
- added TP_VP_0: VP_0, MeasurementPoints:Measurement_Point_Round-SMD-Pad_Small, symbol conn:TEST_1P
- added TP_VP_1: VP_1, MeasurementPoints:Measurement_Point_Round-SMD-Pad_Small, symbol conn:TEST_1P
- C1, C11, C4, C8: footprint Capacitors_SMD:C_0603 -> Capacitor_SMD:C_0805_2012Metric; symbol CP1_Small -> din_meter_atm90e26-rescue:CP1_Small; PN (none) -> C
- C10, C12, C2, C3, C5, C9: value 100n -> .1u; footprint Capacitors_SMD:C_0402 -> Capacitor_SMD:C_0805_2012Metric; symbol C_Small -> din_meter_atm90e26-rescue:C_Small; PN (none) -> C
- C13, C14, C7: footprint Capacitors_SMD:C_0402 -> Capacitor_SMD:C_0805_2012Metric; symbol C_Small -> din_meter_atm90e26-rescue:C_Small; PN (none) -> CC0805JRNPO9BN200
- C15, C16, C17, C18, C19, C20: value 33n -> .033u; footprint Capacitors_SMD:C_0402 -> Capacitor_SMD:C_0805_2012Metric; symbol C_Small -> din_meter_atm90e26-rescue:C_Small; PN (none) -> C
- C6: footprint Capacitors_SMD:C_0402 -> Capacitor_SMD:C_0805_2012Metric; symbol C_Small -> din_meter_atm90e26-rescue:C_Small; PN (none) -> CC0805JRNPO9BN200; manf# GRM1555C1H200JA01D -> CC0805JRNPO9BN200
- G1: symbol LOGO -> din_meter_atm90e26-rescue:LOGO; PN (none) -> X
- J5: symbol CONN_01X10 -> din_meter_atm90e26-rescue:CONN_01X10; PN (none) -> 52418-1010
- L1, L2: footprint Inductors_SMD:L_0402 -> Inductor_SMD:L_0603_1608Metric; symbol L_Core_Ferrite_Small -> din_meter_atm90e26-rescue:L_Core_Ferrite_Small; PN (none) -> CIB10P100NC
- M1, M2: footprint Housings_SSOP:SSOP-28_5.3x10.2mm_Pitch0.65mm -> Housings:SSOP-28_5.3x10.2mm_Pitch0.65mm; symbol ATM90E26_ATM90E26 -> din_meter_atm90e26-rescue:ATM90E26_ATM90E26; PN (none) -> ATM90E26-YU-B
- R1, R2, R3, R4, R5, R6: footprint Resistors_SMD:R_0402 -> Resistor_SMD:R_0805_2012Metric; symbol R_Small -> din_meter_atm90e26-rescue:R_Small; PN (none) -> R
- SYM1: symbol SYM_Flash_Small -> din_meter_atm90e26-rescue:SYM_Flash_Small; PN (none) -> X
- Y1, Y2: footprint Crystals:Crystal_SMD_5032-2pin_5.0x3.2mm -> Crystal:Crystal_SMD_5032-2Pin_5.0x3.2mm; symbol Crystal_Small -> din_meter_atm90e26-rescue:Crystal_Small; PN (none) -> AA-8.192MAGE-T
Connections:
- net labels added: 3V3_M, GND_M, MISO_M, MOSI_M, SCLK_M
- net labels removed: 3V3_ISO, GND_ISO, I2N_0, I2N_0_IN, I2N_1, I2N_1_IN, I2P_0, I2P_0_IN, I2P_1, I2P_1_IN, SCLK, SI/RX, SO/TX
- wire segments 246 -> 217
Other:
- note added: "SPI debug header"
- moved on the sheet: C1, C2, C8, C9
