File: din_meter_atm90e26.kicad_pcb (KiCad board)
At the start: 2 copper layers, 32 x 35.5 mm, 45 parts, among them J1 PCIx1, J2 Conn_01x05, J5 CONN_01X10, M1 ATM90E26_ATM90E26, M2 ATM90E26_ATM90E26, Y1 Crystal_Small, Y2 Crystal_Small

Commit message: updated readme.
Parts:
- J1: value PCIx1 -> PCI_Express; footprint Connectors:PCI-EXPRESS -> FitHome_conn:PCI-EXPRESS
- moved TP_I1P_1 8.10 mm to (136.2, 74.8)
- moved TP_I1N_1 4.56 mm to (136.1, 77.5)
- moved R6 0.92 mm to (139.3, 81.6)
- moved C20 0.63 mm to (137.3, 81.6)
Connections:
- J1 pad A1: 3V3_M -> (no net)
- J1 pad A16: (no net) -> I1N_0_IN
- J1 pad A17: 3V3_CPU -> I1P_0_IN
- J1 pad A18: GND_CPU -> (no net)
- J1 pad A4: (no net) -> I1N_1_IN
- J1 pad A8: GND_M -> I1P_1_IN
- J1 pad B1: VP_1 -> (no net)
- J1 pad B15: I1N_0_IN -> (no net)
- J1 pad B16: (no net) -> GND_CPU
- J1 pad B17: I1P_0_IN -> 3V3_CPU
- J1 pad B2: (no net) -> 3V3_M
- J1 pad B3: I1N_1_IN -> (no net)
- J1 pad B4: I1P_1_IN -> GND_M
- J1 pad B6: (no net) -> VP_1
- J5 pad 1: 3V3_CPU -> GND_CPU
- J5 pad 2: GND_CPU -> 3V3_CPU
Routing:
- net 3V3_CPU: track 38.3 -> 42.7 mm
- net GND_M: track 46.4 -> 42.1 mm
- net I1P_1_IN: track 6.59 -> 3.71 mm
- net GND_CPU: track 41.6 -> 39.1 mm
- net VP_1: track 18.2 -> 16.1 mm, vias 3 -> 4
- net I1N_1: track 14.9 -> 13.0 mm
- net I1N_1_IN: track 5.61 -> 4.23 mm
- net CS_0: track 21.9 -> 20.8 mm
- net 3V3_M: track 40.6 -> 41.5 mm
- net I1P_1: track 18.7 -> 18.1 mm
- net I1P_0_IN: track 3.25 -> 3.75 mm
- net VP_0: vias 2 -> 3

Commit message: OSH Park Rev B
Other:
- board text added: "FirHome Meter Rev B 04/08/2019"
- board text added: "Thanks To"
- board text removed: "FirHome Meter v. A 03/25/2019"
- board text removed: "Thanks to"
Changed lines of the file:
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@@
     (0 F.Cu mixed)
     (31 B.Cu mixed)
-    (32 B.Adhes user hide)
-    (33 F.Adhes user hide)
-    (34 B.Paste user hide)
-    (35 F.Paste user hide)
-    (36 B.SilkS user hide)
+    (32 B.Adhes user)
+    (33 F.Adhes user)
+    (34 B.Paste user)
+    (35 F.Paste user)
+    (36 B.SilkS user)
     (37 F.SilkS user hide)
     (38 B.Mask user hide)
@@
       (net 21 VP_1))
   )
-  (gr_text "FirHome Meter v. A\n03/25/2019" (at 145.31 74.35) (layer B.SilkS)
-    (effects (font (size 0.6 0.6) (thickness 0.15)) (justify mirror))
-  )
-  (gr_text "Thanks to" (at 152.86 63.41) (layer B.SilkS)
-    (effects (font (size 1.5 1.5) (thickness 0.3)))
+  (gr_text "Thanks To" (at 152.53 62.13) (layer B.SilkS)
+    (effects (font (size 1.5 1.5) (thickness 0.3)) (justify mirror))
+  )
+  (gr_text "FirHome Meter Rev B\n04/08/2019" (at 147.32 73.9) (layer B.SilkS)
+    (effects (font (size 1 1) (thickness 0.15)) (justify mirror))
   )
   (gr_line (start 129.9 59.76) (end 129.9 59.62) (layer Edge.Cuts) (width 0.15))
